File: ws2812_boost_driver.kicad_pcb (KiCad board)
At the start: 2 copper layers, 20.5 x 16.5 mm, 21 parts, among them J1 Conn_01x01, J2 Conn_01x01, J3 Conn_01x01, J4 Conn_01x01, J5 Conn_01x01, J6 Conn_01x01, J7 Conn_01x01, J8 Conn_ARM_JTAG_SWD_10, U1 ATSAMD21E15L-A, U2 TC2014-3.3VxCTTR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

Commit message: Add attiny10 hardware spi->ws2812 support
Parts:
- added R7: 10kR, Resistor_SMD:R_0805_2012Metric, F.Cu at (146.6, 91.3)
- added REF**: Logo_WM, Symbol:Logo_WM, B.Cu at (132.9, 101.9)
- added U4: ATtiny10-TS, Package_TO_SOT_SMD:SOT-23-6, F.Cu at (147.5, 95.8)
- moved J3 3.00 mm to (149.0, 99.0)
- moved J5 2.00 mm to (146.0, 102.0)
Connections:
- U1 pad 17: (no net) -> MOSI
- U1 pad 18: (no net) -> SCK
- U1 pad 19: D2 -> (no net)
- U1 pad 20: D1 -> (no net)
- U1 pad 23: (no net) -> D2
- U1 pad 24: DOUT -> D1
Routing:
- net +5V: track 8.29 -> 20.3 mm
- net GND: track 44.3 -> 55.7 mm
- net D1: track 8.98 -> 14.6 mm, vias 0 -> 2
- net DOUT: track 6.82 -> 2.47 mm
- net SCK: track 0.00 -> 4.14 mm
- net Net-(R7-Pad2): track 0.00 -> 3.39 mm
- net MOSI: track 0.00 -> 3.11 mm
- net D2: track 7.45 -> 10.5 mm, vias 0 -> 2
- net RESET: track 21.2 -> 20.3 mm
Other:
- board text added: "11/13/20"
- board text added: "v0.0.0"
